Commit message: Legs finished. First control attempts

File: spider_description/macros/macros.xacro (robot description, xacro)
@@ -19,8 +19,8 @@
   />
 </macro>
-<macro name="make_leg" params="name reflect parent">
+<macro name="make_leg" params="name reflect parent xpos">
   <link name="${name}_a_servo">
     <collision>
-      <origin xyz="0 0 0" rpy="0 1.57 0"/>
+      <origin xyz="0 0 0" rpy="0 0 0"/>
       <geometry>
         <box size="${servo_length} ${servo_width} ${servo_height}"/>
@@ -28,12 +28,12 @@
     </collision>
     <visual>
-      <origin xyz="0 0 0" rpy="0 1.57 0"/>
+      <origin xyz="0 0 0" rpy="0 0 0"/>
       <geometry>
         <box size="${servo_length} ${servo_width} ${servo_height}"/>
       </geometry>
-      <material name="white"/>
+      <material name="blue"/>
     </visual>
     <inertial>
-      <origin xyz="0 0 0" rpy="0 1.57 0"/>
+      <origin xyz="0 0 0" rpy="0 0 0"/>
       <mass value="${servo_mass}"/>
       <box_inertia m="${servo_mass}" x="${servo_length}" y="${servo_width}" z="${servo_height}"/>
@@ -42,5 +42,5 @@
   <link name="${name}_b_servo">
     <collision>
-      <origin xyz="0 0 0" rpy="1.57 0 ${reflect*1.57}"/>
+      <origin xyz="0 0 0" rpy="0 0 0"/>
       <geometry>
         <box size="${servo_length} ${servo_width} ${servo_height}"/>
@@ -48,5 +48,5 @@
     </collision>
     <visual>
-      <origin xyz="0 0 0" rpy="1.57 0 ${reflect*1.57}"/>
+      <origin xyz="0 0 0" rpy="0 0 0"/>
       <geometry>
         <box size="${servo_length} ${servo_width} ${servo_height}"/>
@@ -55,5 +55,5 @@
     </visual>
     <inertial>
-      <origin xyz="0 0 0" rpy="1.57 0 ${reflect*1.57}"/>
+      <origin xyz="0 0 0" rpy="0 0 0"/>
       <mass value="${servo_mass}"/>
       <box_inertia m="${servo_mass}" x="${servo_length}" y="${servo_width}" z="${servo_height}"/>
@@ -103,28 +103,58 @@
     <parent link="body"/>
     <child link="${name}_a_servo"/>
-    <origin xyz="0 ${reflect*(body_width+servo_length)/2} 0" rpy="0 0 ${reflect*1.57}"/>
+    <origin xyz="${xpos} ${(-1)*((body_width+servo_length)/2)*(2*reflect-1)} 0" rpy="0 -1.57 ${(-1)*(1.57)*(2*reflect-1)}"/>
   </joint>
   <joint name="${name}_a_joint" type="revolute">
     <parent link="${name}_a_servo"/>
     <child link="${name}_b_servo"/>
-    <origin xyz="0 0 ${servo_height/2}" rpy="0 0 0"/>
-    <axis xyz="0 0 1"/>
-    <limit lower="${reflect*1.57}" upper="${reflect*-1.57}" effort="1" velocity="10"/>
+    <origin xyz="${(servo_length+servo_width)/2} 0 ${-servo_height/4}" rpy="0 0 ${(1.57)*(2*reflect-1)}"/>
+    <axis xyz="0 1 0"/>
+    <limit lower="-1.57" upper="1.57" effort="1" velocity="1"/>
   </joint>
   <joint name="${name}_b_joint" type="revolute">
     <parent link="${name}_b_servo"/>
     <child link="${name}_proximal_leg"/>
-    <origin xyz="0 ${reflect*(servo_width+leg_radius)} 0" rpy="0 0 0"/>
-    <axis xyz="0 1 0"/>
-    <!-- Aquí está el problema. Para un lado debe ser l=-3.14 y u=0 y para el otro l=0 y u=3.14 -->
-    <limit lower="0" upper="${reflect*3.14}" effort="1" velocity="10"/>
+    <origin xyz="${(servo_length+leg_radius)/2} 0 ${-servo_height/4}" rpy="${(1.57)*(2*reflect-1)} 0 0"/>
+    <axis xyz="1 0 0"/>
+    <!-- Aqui esta el problema. Para un lado debe ser l=-3.14 y u=0 y para el otro l=0 y u=3.14 -->
+    <limit lower="${(1-reflect)*(-3.14)+(reflect)*(0)}" upper="${(1-reflect)*(0)+(reflect)*(3.14)}" effort="1" velocity="1"/>
   </joint>
   <joint name="${name}_c_joint" type="revolute">
     <parent link="${name}_proximal_leg"/>
     <child link="${name}_distal_leg"/>
-    <origin xyz="0 ${reflect*(leg_radius*2)} ${leg_a_length}" rpy="0 3.14 0"/>
-    <axis xyz="0 1 0"/>
-    <limit lower="-3.14" upper="0" effort="1" velocity="10"/>
+    <origin xyz="0 ${(-1)*(2*reflect-1)*(leg_radius*2)} ${leg_a_length}" rpy="0 3.14 0"/>
+    <axis xyz="1 0 0"/>
+    <limit lower="${(1-reflect)*(-3.14)+(reflect)*(0)}" upper="${(1-reflect)*(0)+(reflect)*(3.14)}" effort="1" velocity="1"/>
   </joint>
+  <transmission name="${name}_a_transmission">
+    <type>transmission_interface/SimpleTransmission</type>
+    <joint name="${name}_a_joint">
+      <hardwareInterface>PositionJointInterface</hardwareInterface>
+    </joint>
+    <actuator name="${name}_a_joint_leg_actuator">
+      <hardwareInterface>PositionJointInterface</hardwareInterface>
+      <mechanicalReduction>10</mechanicalReduction>
+    </actuator>
+  </transmission>
+  <transmission name="${name}_b_transmission">
+    <type>transmission_interface/SimpleTransmission</type>
+    <joint name="${name}_b_joint">
+      <hardwareInterface>PositionJointInterface</hardwareInterface>
+    </joint>
+    <actuator name="${name}_b_joint_leg_actuator">
+      <hardwareInterface>PositionJointInterface</hardwareInterface>
+      <mechanicalReduction>10</mechanicalReduction>
+    </actuator>
+  </transmission>
+  <transmission name="${name}_c_transmission">
+    <type>transmission_interface/SimpleTransmission</type>
+    <joint name="${name}_c_joint">
+      <hardwareInterface>PositionJointInterface</hardwareInterface>
+    </joint>
+    <actuator name="${name}_c_joint_leg_actuator">
+      <hardwareInterface>PositionJointInterface</hardwareInterface>
+      <mechanicalReduction>10</mechanicalReduction>
+    </actuator>
+  </transmission>
 </macro>
 </robot>

File: spider_description/urdf/spider.xacro (robot description, xacro)
@@ -18,4 +18,8 @@
 <!-- Links -->
 <link name="base_link"/>
+<make_leg name="FL" reflect="0" parent="body" xpos="${body_length/4}"/>
+<make_leg name="FR" reflect="1" parent="body" xpos="${body_length/4}"/>
+<make_leg name="BL" reflect="0" parent="body" xpos="${-body_length/4}"/>
+<make_leg name="BR" reflect="1" parent="body" xpos="${-body_length/4}"/>
 <link name="body">
 	<collision>
@@ -38,176 +42,7 @@
 	</inertial>
 </link>
-<link name="a_servo">
-	<collision>
-		<origin xyz="0 0 0" rpy="0 1.57 3.14"/>
-		<geometry>
-			<box size="${servo_length} ${servo_width} ${servo_height}"/>
-		</geometry>
-	</collision>
-	<visual>
-		<origin xyz="0 0 0" rpy="0 1.57 3.14"/>
-		<geometry>
-			<box size="${servo_length} ${servo_width} ${servo_height}"/>
-		</geometry>
-		<material name="white"/>
-	</visual>
-	<inertial>
-		<origin xyz="0 0 0" rpy="0 1.57 3.14"/>
-		<mass value="${servo_mass}"/>
-		<box_inertia m="${servo_mass}" x="${servo_length}" y="${servo_width}" z="${servo_height}"/>
-	</inertial>
-</link>
-<link name="b_servo">
-	<collision>
-		<origin xyz="0 0 0" rpy="1.57 0 -1.57"/>
-		<geometry>
-			<box size="${servo_length} ${servo_width} ${servo_height}"/>
-		</geometry>
-	</collision>
-	<visual>
-		<origin xyz="0 0 0" rpy="1.57 0 -1.57"/>
-		<geometry>
-			<box size="${servo_length} ${servo_width} ${servo_height}"/>
-		</geometry>
-		<material name="blue"/>
-	</visual>
-	<inertial>
-		<origin xyz="0 0 0" rpy="1.57 0 -1.57"/>
-		<mass value="${servo_mass}"/>
-		<box_inertia m="${servo_mass}" x="${servo_length}" y="${servo_width}" z="${servo_height}"/>
-	</inertial>
-</link>
-<link name="proximal_leg">
-	<collision>
-		<origin xyz="0 0 ${leg_a_length/2}" rpy="0 0 0"/>
-		<geometry>
-			<cylinder length="${leg_a_length}" radius="${leg_radius}"/>
-		</geometry>
-	</collision>
-	<visual>
-		<origin xyz="0 0 ${leg_a_length/2}" rpy="0 0 0"/>
-		<geometry>
-			<cylinder length="${leg_a_length}" radius="${leg_radius}"/>
-		</geometry>
-		<material name="white"/>
-	</visual>
-	<inertial>
-		<origin xyz="0 0 ${leg_a_length/2}" rpy="0 0 0"/>
-		<mass value="${leg_mass}"/>
-		<cylinder_inertia m="${leg_mass}" r="${leg_radius}" h="${leg_a_length}"/>
-	</inertial>
-</link>
-<link name="distal_leg">
-	<collision>
-		<origin xyz="0 0 ${leg_b_length/2}" rpy="0 0 0"/>
-		<geometry>
-			<cylinder length="${leg_b_length}" radius="${leg_radius}"/>
-		</geometry>
-	</collision>
-	<visual>
-		<origin xyz="0 0 ${leg_b_length/2}" rpy="0 0 0"/>
-		<geometry>
-			<cylinder length="${leg_b_length}" radius="${leg_radius}"/>
-		</geometry>
-		<material name="white"/>
-	</visual>
-	<inertial>
-		<origin xyz="0 0 ${leg_b_length/2}" rpy="0 0 0"/>
-		<mass value="${leg_mass}"/>
-		<cylinder_inertia m="${leg_mass}" r="${leg_radius}" h="${leg_b_length}"/>
-	</inertial>
-</link>
-<!-- Joints -->
 <joint name="base_joint" type="fixed">
 	<parent link="base_link"/>
 	<child link="body"/>
 </joint>
-<joint name="leg_fix" type="fixed">
-	<parent link="body"/>
-	<child link="a_servo"/>
-	<origin xyz="0 ${(body_width+servo_length)/2} 0" rpy="0 0 1.57"/>
-</joint>
-<make_leg name="FL" reflect="-1" parent="body"/>
-<joint name="a_joint" type="revolute">
-	<parent link="a_servo"/>
-	<child link="b_servo"/>
-	<origin xyz="0 0 ${servo_height/2}" rpy="0 0 0"/>
-	<axis xyz="0 0 1"/>
-	<limit lower="-1.57" upper="1.57" effort="1" velocity="10"/>
-</joint>
-<joint name="b_joint" type="revolute">
-	<parent link="b_servo"/>
-	<child link="proximal_leg"/>
-	<origin xyz="0 ${servo_width+leg_radius} 0" rpy="0 0 0"/>
-	<axis xyz="0 1 0"/>
-	<limit lower="0" upper="3.14" effort="1" velocity="10"/>
-</joint>
-<joint name="c_joint" type="revolute">
-	<parent link="proximal_leg"/>
-	<child link="distal_leg"/>
-	<origin xyz="0 ${leg_radius*2} ${leg_a_length}" rpy="0 3.14 0"/>
-	<axis xyz="0 1 0"/>
-	<limit lower="-3.14" upper="0" effort="1" velocity="10"/>
-</joint>
-<!-- Transmissions -->
-<transmission name="transmission_a">
-	<type>transmission_interface/SimpleTransmission</type>
-	<joint name="a_joint">
-		<hardwareInterface>PositionJointInterface</hardwareInterface>
-	</joint>
-	<actuator name="a_joint_leg_actuator">
-		<hardwareInterface>PositionJointInterface</hardwareInterface>
-		<mechanicalReduction>10</mechanicalReduction>
-	</actuator>
-</transmission>
-<transmission name="transmission_b">
-	<type>transmission_interface/SimpleTransmission</type>
-	<joint name="b_joint">
-		<hardwareInterface>PositionJointInterface</hardwareInterface>
-	</joint>
-	<actuator name="b_joint_leg_actuator">
-		<hardwareInterface>PositionJointInterface</hardwareInterface>
-		<mechanicalReduction>10</mechanicalReduction>
-	</actuator>
-</transmission>
-<transmission name="transmission_c">
-	<type>transmission_interface/SimpleTransmission</type>
-	<joint name="c_joint">
-		<hardwareInterface>PositionJointInterface</hardwareInterface>
-	</joint>
-	<actuator name="c_joint_leg_actuator">
-		<hardwareInterface>PositionJointInterface</hardwareInterface>
-		<mechanicalReduction>10</mechanicalReduction>
-	</actuator>
-</transmission>
-<transmission name="FL_a_transmission">
-	<type>transmission_interface/SimpleTransmission</type>
-	<joint name="FL_a_joint">
-		<hardwareInterface>PositionJointInterface</hardwareInterface>
-	</joint>
-	<actuator name="FL_a_joint_leg_actuator">
-		<hardwareInterface>PositionJointInterface</hardwareInterface>
-		<mechanicalReduction>10</mechanicalReduction>
-	</actuator>
-</transmission>
-<transmission name="FL_b_transmission">
-	<type>transmission_interface/SimpleTransmission</type>
-	<joint name="FL_b_joint">
-		<hardwareInterface>PositionJointInterface</hardwareInterface>
-	</joint>
-	<actuator name="FL_b_joint_leg_actuator">
-		<hardwareInterface>PositionJointInterface</hardwareInterface>
-		<mechanicalReduction>10</mechanicalReduction>
-	</actuator>
-</transmission>
-<transmission name="FL_c_transmission">
-	<type>transmission_interface/SimpleTransmission</type>
-	<joint name="FL_c_joint">
-		<hardwareInterface>PositionJointInterface</hardwareInterface>
-	</joint>
-	<actuator name="FL_c_joint_leg_actuator">
-		<hardwareInterface>PositionJointInterface</hardwareInterface>
-		<mechanicalReduction>10</mechanicalReduction>
-	</actuator>
-</transmission>
 </robot>

Commit message: Before I begin screwing things up.

File: spider_description/macros/macros.xacro (robot description, xacro)
@@ -110,5 +110,5 @@
     <origin xyz="${(servo_length+servo_width)/2} 0 ${-servo_height/4}" rpy="0 0 ${(1.57)*(2*reflect-1)}"/>
     <axis xyz="0 1 0"/>
-    <limit lower="-1.57" upper="1.57" effort="1" velocity="1"/>
+    <limit lower="-1.57" upper="1.57" effort="1" velocity="3"/>
   </joint>
   <joint name="${name}_b_joint" type="revolute">
@@ -118,5 +118,5 @@
     <axis xyz="1 0 0"/>
     <!-- Aqui esta el problema. Para un lado debe ser l=-3.14 y u=0 y para el otro l=0 y u=3.14 -->
-    <limit lower="${(1-reflect)*(-3.14)+(reflect)*(0)}" upper="${(1-reflect)*(0)+(reflect)*(3.14)}" effort="1" velocity="1"/>
+    <limit lower="${(1-reflect)*(-3.14)+(reflect)*(0)}" upper="${(1-reflect)*(0)+(reflect)*(3.14)}" effort="1" velocity="3"/>
   </joint>
   <joint name="${name}_c_joint" type="revolute">
@@ -125,5 +125,5 @@
     <origin xyz="0 ${(-1)*(2*reflect-1)*(leg_radius*2)} ${leg_a_length}" rpy="0 3.14 0"/>
     <axis xyz="1 0 0"/>
-    <limit lower="${(1-reflect)*(-3.14)+(reflect)*(0)}" upper="${(1-reflect)*(0)+(reflect)*(3.14)}" effort="1" velocity="1"/>
+    <limit lower="${(1-reflect)*(-3.14)+(reflect)*(0)}" upper="${(1-reflect)*(0)+(reflect)*(3.14)}" effort="1" velocity="3"/>
   </joint>
   <transmission name="${name}_a_transmission">

File: spider_description/urdf/spider.xacro (robot description, xacro)
@@ -7,5 +7,5 @@
 <xacro:property name="leg_b_length" value="0.12"/>
 <xacro:property name="leg_radius" value="0.005"/>
-<xacro:property name="leg_mass" value="0.1"/>
+<xacro:property name="leg_mass" value="0.05"/>
 <xacro:property name="servo_length" value="0.02"/>
 <xacro:property name="servo_width" value="0.01"/>
@@ -18,8 +18,4 @@
 <!-- Links -->
 <link name="base_link"/>
-<make_leg name="FL" reflect="0" parent="body" xpos="${body_length/4}"/>
-<make_leg name="FR" reflect="1" parent="body" xpos="${body_length/4}"/>
-<make_leg name="BL" reflect="0" parent="body" xpos="${-body_length/4}"/>
-<make_leg name="BR" reflect="1" parent="body" xpos="${-body_length/4}"/>
 <link name="body">
 	<collision>
@@ -42,4 +38,10 @@
 	</inertial>
 </link>
+<make_leg name="FL" reflect="0" parent="body" xpos="${body_length/2}"/>
+<make_leg name="FR" reflect="1" parent="body" xpos="${body_length/2}"/>
+<make_leg name="ML" reflect="0" parent="body" xpos="${0}"/>
+<make_leg name="MR" reflect="1" parent="body" xpos="${0}"/>
+<make_leg name="BL" reflect="0" parent="body" xpos="${-body_length/2}"/>
+<make_leg name="BR" reflect="1" parent="body" xpos="${-body_length/2}"/>
 <joint name="base_joint" type="fixed">
 	<parent link="base_link"/>
