Commit message: Genetic learning almost working. Need for some inertial fixes.

File: spider_description/macros/leg.xacro (robot description, xacro)
@@ -122,4 +122,13 @@
     </actuator>
   </transmission>
+  <gazebo reference="${name}_distal_leg">
+    <mu1 value="10.0" />
+    <mu2 value="1.0" />
+    <fdir1 value="1 0 0"/>
+    <kp value="1000000.0"/>
+    <kd value="100.0"/>
+    <material>Gazebo/Black</material>
+    <turnGravityOff>false</turnGravityOff>
+  </gazebo>
 </macro>
 </robot>
