Commit message: First attempts to automate the gait testing

File: spider_description/urdf/spider.xacro (robot description, xacro)
@@ -3,5 +3,6 @@
 <xacro:include filename="$(find spider_description)/materials/materials.xacro" />
 <xacro:include filename="$(find spider_description)/urdf/spider.gazebo" />
-<xacro:include filename="$(find spider_description)/macros/macros.xacro" />
+<xacro:include filename="$(find spider_description)/macros/inertia.xacro" />
+<xacro:include filename="$(find spider_description)/macros/leg.xacro" />
 <xacro:property name="leg_a_length" value="0.07"/>
 <xacro:property name="leg_b_length" value="0.12"/>
@@ -11,9 +12,11 @@
 <xacro:property name="servo_width" value="0.01"/>
 <xacro:property name="servo_height" value="0.03"/>
-<xacro:property name="servo_mass" value="0.009"/>
+<xacro:property name="servo_mass" value="0.1"/>
 <xacro:property name="body_length" value="0.15"/>
 <xacro:property name="body_width" value="0.10"/>
 <xacro:property name="body_height" value="0.05"/>
 <xacro:property name="body_mass" value="0.5"/>
+<xacro:property name="servo_effort" value="1000"/>
+<xacro:property name="servo_velocity" value="3"/>
 <!-- Links -->
 <link name="base_link"/>
@@ -32,9 +35,5 @@
 		<material name="white"/>
 	</visual>
-	<inertial>
-		<origin xyz="0 0 0" rpy="0 0 0"/>
-		<mass value="${body_mass}"/>
-		<box_inertia m="${body_mass}" x="${body_length}" y="${body_width}" z="${body_height}"/>
-	</inertial>
+	<xacro:box_inertial m="${body_mass}" x="${body_length}" y="${body_width}" z="${body_height}"/>
 </link>
 <make_leg name="FL" reflect="0" parent="body" xpos="${body_length/2}"/>
